File: jeff_board_kicad/VAP_thermal_control.sch (KiCad schematic (older format))
At the start: 27 parts, among them J1 Conn_01x02_Female, J2 Conn_01x02_Female, J3 Conn_01x02_Female, Q1 IRLB8721PBF, Q2 IRLB8721PBF, U1 TSR_1-24150, U2 MAX31865Breakout, U3 MLX90614, U4 MIC4427

Commit message: Prelim Layout of jeff V2
Added two channels of PWM, so we can drive 4 of (Fan/Heater/LEDs).
Parts:
- added C10: 0.1u, Capacitors_THT:CP_Radial_D5.0mm_P2.00mm, symbol Device:CP
- added C11: 1u, Capacitors_THT:CP_Radial_D5.0mm_P2.00mm, symbol Device:CP
- added D3, D4: LED, LEDs:LED_D5.0mm, symbol Device:LED
- added J4, J5: Conn_01x02_Female, Connectors_Phoenix:PhoenixContact_MSTBVA-G_02x5.00mm_Vertical, symbol Connector:Conn_01x02_Female
- added Q3, Q4: IRLB8721PBF, TO_SOT_Packages_THT:TO-220-3_Vertical, symbol Transistor_FET:IRLB8721PBF
- added R10, R9: 10k, Resistors_SMD:R_0805_HandSoldering, symbol Device:R
- added R7, R8: 1k, Resistors_SMD:R_0805_HandSoldering, symbol Device:R
- added U5: MIC4427, Housings_DIP:DIP-8_W7.62mm, symbol Driver_FET:MIC4427
- J1, J2, J3: footprint Wire_Pads:SolderWirePad_2x_2mmDrill -> Connectors_Phoenix:PhoenixContact_MSTBVA-G_02x5.00mm_Vertical
Connections:
- net +24V: now also J4.1 (Pin_1), J5.1 (Pin_1), R7.1, R8.1
- net +5V: now also A1.30 (VIN), C10.1, C11.1, U5.6 (V+); no longer A1.27 (+5V)
- net GND: now also A1.29 (GND), A1.4 (GND), C10.2, C11.2, Q3.3 (S), Q4.3 (S), R10.1, R9.1, U5.3 (GND)
- net at A1.12 (D9): now also R3.1, U4.4 (IN_B)
- net at A1.8 (D5): now also R10.2, U5.4 (IN_B)
- new net: A1.6 (D3), R9.2, U5.2 (IN_A)
- new net: Q3.1 (G), U5.5 (OUT_B)
- new net: Q4.1 (G), U5.7 (OUT_A)
- new net: D3.1 (K), J4.2 (Pin_2), Q3.2 (D)
- new net: D4.1 (K), J5.2 (Pin_2), Q4.2 (D)
- new net: D3.2 (A), R7.2
- new net: D4.2 (A), R8.2
- no-connect marks 0 -> 16
Other:
- moved on the sheet: C5
